File: eagle files/32u4_macropad.sch (EAGLE design)
At the start: 63 parts, among them IC1 IS31FL3733-TQLS4, J1 TYPE-C-31-M-12, Q2 16Mhz, SW2 SWITCH-SMD-EVP-BB2A9B00, U1 ATMEGA32U4-TQFP44

Commit message: Added underglow WS2812B LEDs
Parts:
- removed D1, D10, D11, D12, D13, D14, D15, D16, D2, D3, D4, D5, D7, D8, D9: (no value), Components:DIODE-SOD-123
- removed F1, F10, F11, F12, F2, F3, F4, F5, F6, F7, F8, F9, U$3, U$4, U$5: KEYSWITCH-PLAIN-MX-1U, Keyboard:KEYSWITCH-PLAIN-MX-1U
- added C15: 0.47uF, Components:CAPACITOR-0603
- added C16, C17: 100uF, Components:CAPACITOR-0603
- added LED1, LED2, LED3, LED4: WS2812B5050, WS2812B:WS2812B5050
- C14: value 0.1uF -> 100uF
- C8: value 0.47uF -> 100uF
- U$2: value KEYSWITCH-PLAIN-MX-1U -> KEYSWITCH-RGBSMDLED-MX-1U-SMDRGB; device Keyboard:KEYSWITCH-PLAIN-MX-1U -> Keyboard:KEYSWITCH-RGBSMDLED-MX-1U-SMDRGB
Connections:
- removed net AVCC: C14.2, C8.2, IC1.AVCC
- removed net DVCC: IC1.DVCC
- removed net INTB??: R9.1
- removed net N$11: D12.A, F12.P0
- removed net N$12: D11.A, U$2.P0
- removed net N$13: D14.A, U$5.P0
- removed net N$14: D15.A, F8.P0
- removed net N$23: D10.A, U$4.P0
- removed net N$25: D2.A, U$3.P0
- removed net N$28: C5.2
- removed net N$9: D1.A, F10.P0
- removed net PVCC_1: C7.2, IC1.PVCC_1
- removed net PVCC_2: C3.2, C4.2, IC1.PVCC_2
- removed net USE??: IC1.INTB
- new net INTBUSE??: IC1.INTB, R9.1
- new net UNDGLOW: LED1.DI, U1.PF1(ADC1)
- net 0: now also C15.1, C16.1, C17.1, IC1.AGND, IC1.PGND_1, IC1.PGND_2, LED1.GND, LED2.GND, LED3.GND, LED4.GND
- net C0: no longer F1.P1, F5.P1, F9.P1
- net C1: no longer F10.P1, F2.P1, F6.P1, U$3.P1
- net C2: no longer F11.P1, F12.P1, F3.P1, F7.P1
- net C3: no longer F4.P1, F8.P1, U$4.P1, U$5.P1
- net N$1: now also U$2.P0; no longer F1.P0
- net N$10: now also C16.2, LED3.VDD; no longer D13.A, F11.P0
- net N$2: now also U$2.R-; no longer D3.A, F2.P0
- net N$3: now also U$2.G-; no longer D4.A, F3.P0
- net N$4: now also U$2.B-; no longer D5.A, F4.P0
- net N$5: now also LED1.DO, LED2.DI; no longer D7.A, F5.P0
- net N$6: now also LED3.DO, LED4.DI; no longer D9.A, F6.P0
- net N$7: now also LED2.DO, LED3.DI; no longer D16.A, F7.P0
- net N$8: now also C14.2, LED2.VDD; no longer D8.A, F9.P0
- net R0: no longer D3.C, D4.C, D5.C, D6.C
- net R1: no longer D15.C, D16.C, D7.C, D9.C
- net R2: no longer D1.C, D13.C, D14.C, D8.C
- net R3: no longer D10.C, D11.C, D12.C, D2.C
- net VCC: now also C15.2, C17.2, C3.2, C4.2, C5.2, C7.2, C8.2, IC1.AVCC, IC1.DVCC, IC1.PVCC_1, IC1.PVCC_2, IC1.VIO, LED1.VDD, LED4.VDD
Other:
- note added: "MCU"
- note added: "UNDERGLOW"
- moved on the sheet: C1, C10, C11, C12, C13, C14, C2, C3, C4, C5, C6, C7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

Commit message: New SK6812MINI-E footprint, added ground pin on crystal, fixed misconnections
Parts:
- removed C14, C16, C17, C8: 100uF, Components:CAPACITOR-0603
- removed LED1, LED2, LED3, LED4: WS2812B5050, WS2812B:WS2812B5050
- removed Q2: 16Mhz, crystal-geyer_V1_0:KX-5
- added C18, C19, C20, C21: 100uF, Components:CAPACITOR-0603
- added D0, D1, D10, D11, D12, D13, D14, D15, D2, D3, D4, D5, D7, D8, D9: (no value), Components:DIODE-SOD-123
- added Q1: 16Mhz, crystal-geyer_V1_0_NIC:KX-5
- added U$1, U$10, U$11, U$12, U$13, U$14, U$15, U$16, U$3, U$4, U$5, U$6, U$7, U$8, U$9: KEYSWITCH-PLAIN-MX-1U, Keyboard:KEYSWITCH-PLAIN-MX-1U
- added U$17, U$18, U$19, U$20: SK6812MINI-E, SK:SK6812MINI-E
- U$2: value KEYSWITCH-RGBSMDLED-MX-1U-SMDRGB -> KEYSWITCH-PLAIN-MX-1U; device Keyboard:KEYSWITCH-RGBSMDLED-MX-1U-SMDRGB -> Keyboard:KEYSWITCH-PLAIN-MX-1U
Connections:
- net C2 renamed C2SWTC
- removed net C0: U$2.P1, U1.PC6(OC3A/!OC4A)
- removed net C1: U1.PC7(ICP3/CLK0/OC4A)
- removed net C3: U1.PD3(TXD1/INT3)
- removed net N$10: C16.2, LED3.VDD
- removed net N$18: SW2.2
- removed net N$2 (its old number): U$2.R-
- removed net N$24: C2.2, Q2.1, U1.XTAL2
- removed net N$7: LED2.DO, LED3.DI
- removed net N$8: C14.2, LED2.VDD
- removed net R0: U1.PD4(ICP1/ADC8)
- removed net R1: U1.PD5(XCLK1/!CTS)
- removed net R2: U1.PD6(T1/ADC9/!OC4D)
- removed net R3: U1.PD7(T0/OC4D/ADC10)
- new net C0RGB: IC1.CS1
- new net C0SWTCH: U$1.P1, U$16.P1, U$8.P1, U$9.P1, U1.PC6(OC3A/!OC4A)
- new net C1RGB: IC1.CS2
- new net C1SWTCH: U$10.P1, U$15.P1, U$2.P1, U$7.P1, U1.PC7(ICP3/CLK0/OC4A)
- new net C2RGB: IC1.CS3
- new net C2SWTCH: U$11.P1, U$14.P1, U$3.P1, U$6.P1
- new net C3RGB: IC1.CS4
- new net C3SWTCH: U$12.P1, U$13.P1, U$4.P1, U$5.P1, U1.PD3(TXD1/INT3)
- new net N$12: D6.A, U$6.P0
- new net N$13: D9.A, U$10.P0
- new net N$23: D10.A, U$11.P0
- new net N$25: U$18.DIN, U$19.DOUT
- new net N$28: D3.A, U$4.P0
- new net N$29: D7.A, U$5.P0
- new net N$30: D11.A, U$12.P0
- new net N$31: D13.A, U$15.P0
- new net N$32: D14.A, U$14.P0
- new net N$33: D12.A, U$16.P0
- new net N$34: D15.A, U$13.P0
- new net N$36: C18.2, C19.2, C20.2, C21.2, U$17.VDD, U$18.VDD, U$19.VDD, U$20.VDD
- new net N$38: D8.A, U$9.P0
- new net N$39: U$19.DIN, U$20.DOUT
- new net N$9: D4.A, U$8.P0
- new net R0BLUE: IC1.SW10
- new net R0GREEN: IC1.SW11
- new net R0RED: IC1.SW12
- new net R0SWTCH: D0.C, D1.C, D2.C, D3.C, D5.A, U$7.P0, U1.PD4(ICP1/ADC8)
- new net R1BLUE: IC1.SW7
- new net R1GREEN: IC1.SW8
- new net R1RED: IC1.SW9
- new net R1SWTCH: D4.C, D5.C, D6.C, D7.C, U1.PD5(XCLK1/!CTS)
- new net R2BLUE: IC1.SW4
- new net R2GREEN: IC1.SW5
- new net R2RED: IC1.SW6
- new net R2SWTCH: D10.C, D11.C, D8.C, D9.C, U1.PD6(T1/ADC9/!OC4D)
- new net R3BLUE: IC1.SW1
- new net R3GREEN: IC1.SW2
- new net R3RED: IC1.SW3
- new net R3SWTCH: D12.C, D13.C, D14.C, D15.C, U1.PD7(T0/OC4D/ADC10)
- net 0: now also C18.1, C19.1, C20.1, C21.1, Q1.P$1, U$17.GND, U$18.GND, U$19.GND, U$20.GND; no longer C14.1, C16.1, C17.1, C8.1, LED1.GND, LED2.GND, LED3.GND, LED4.GND
- net N$1: now also D0.A, U$1.P0; no longer D6.A, U$2.P0
- net N$17: now also SW2.2
- net N$21: now also Q1.1; no longer Q2.2
- net N$3: now also D1.A, U$2.P0; no longer U$2.G-
- net N$4: now also D2.A, U$3.P0; no longer U$2.B-
- net N$5: now also C2.2, Q1.2, U1.XTAL2; no longer LED1.DO, LED2.DI
- net N$6: now also U$17.DIN, U$18.DOUT; no longer LED3.DO, LED4.DI
- net UNDGLOW: now also U$20.DIN; no longer LED1.DI
- net VCC: no longer C17.2, C8.2, LED1.VDD, LED4.VDD
Other:
- note added: "SWITCH MATRIX"
- moved on the sheet: C1, C10, C11, C12, C13, C15, C2, C3, C4, C5, C6, C7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

Commit message: started board, added rgb matrix
Parts:
- removed U$1, U$10, U$11, U$12, U$13, U$14, U$15, U$16, U$2, U$3, U$4, U$5, U$6, U$7, U$8, U$9: KEYSWITCH-PLAIN-MX-1U, Keyboard:KEYSWITCH-PLAIN-MX-1U
- added F1, F10, F11, F12, F13, F14, F15, F16, F2, F3, F4, F5, F6, F7, F8, F9: KEYSWITCH-PLAIN-MX-1U, Keyboard:KEYSWITCH-PLAIN-MX-1U
- added LED1, LED10, LED11, LED12, LED13, LED14, LED15, LED16, LED2, LED3, LED4, LED5, LED6, LED7, LED8, LED9: 6028RGBLED_BOTTOM, 6028LED:6028RGBLED_BOTTOM
- added R12: 500, Components:RESISTOR-0603
- U$17, U$18, U$19, U$20: value SK6812MINI-E -> SK6812MINI-E_BOTTOM; device SK:SK6812MINI-E -> SK6812MINI-E:SK6812MINI-E_BOTTOM
Connections:
- removed net C2SWTC: U1.PD2(RXD1/INT2)
- removed net N$36: C18.2, C19.2, C20.2, C21.2, U$17.VDD, U$18.VDD, U$19.VDD, U$20.VDD
- new net N$11: D5.A, F6.P0
- new net N$7: R12.1, U$20.DIN
- net C0RGB: now also LED1.VIN, LED13.VIN, LED5.VIN, LED9.VIN
- net C0SWTCH: now also F1.P1, F13.P1, F5.P1, F9.P1; no longer U$1.P1, U$16.P1, U$8.P1, U$9.P1
- net C1RGB: now also LED10.VIN, LED14.VIN, LED2.VIN, LED6.VIN
- net C1SWTCH: now also F10.P1, F14.P1, F2.P1, F6.P1; no longer U$10.P1, U$15.P1, U$2.P1, U$7.P1
- net C2RGB: now also LED11.VIN, LED15.VIN, LED3.VIN, LED7.VIN
- net C2SWTCH: now also F11.P1, F15.P1, F3.P1, F7.P1, U1.PD2(RXD1/INT2); no longer U$11.P1, U$14.P1, U$3.P1, U$6.P1
- net C3RGB: now also LED12.VIN, LED16.VIN, LED4.VIN, LED8.VIN
- net C3SWTCH: now also F12.P1, F16.P1, F4.P1, F8.P1; no longer U$12.P1, U$13.P1, U$4.P1, U$5.P1
- net N$1: now also F1.P0; no longer U$1.P0
- net N$12: now also F7.P0; no longer U$6.P0
- net N$13: now also F10.P0; no longer U$10.P0
- net N$23: now also F11.P0; no longer U$11.P0
- net N$28: now also F4.P0; no longer U$4.P0
- net N$29: now also F8.P0; no longer U$5.P0
- net N$3: now also F2.P0; no longer U$2.P0
- net N$30: now also F12.P0; no longer U$12.P0
- net N$31: now also F14.P0; no longer U$15.P0
- net N$32: now also F15.P0; no longer U$14.P0
- net N$33: now also F13.P0; no longer U$16.P0
- net N$34: now also F16.P0; no longer U$13.P0
- net N$38: now also F9.P0; no longer U$9.P0
- net N$4: now also F3.P0; no longer U$3.P0
- net N$9: now also F5.P0; no longer U$8.P0
- net R0BLUE: now also LED1.B, LED2.B, LED3.B, LED4.B
- net R0GREEN: now also LED1.G, LED2.G, LED3.G, LED4.G
- net R0RED: now also LED1.R, LED2.R, LED3.R, LED4.R
- net R0SWTCH: no longer D5.A, U$7.P0
- net R1BLUE: now also LED5.B, LED6.B, LED7.B, LED8.B
- net R1GREEN: now also LED5.G, LED6.G, LED7.G, LED8.G
- net R1RED: now also LED5.R, LED6.R, LED7.R, LED8.R
- net R2BLUE: now also LED10.B, LED11.B, LED12.B, LED9.B
- net R2GREEN: now also LED10.G, LED11.G, LED12.G, LED9.G
- net R2RED: now also LED10.R, LED11.R, LED12.R, LED9.R
- net R3BLUE: now also LED13.B, LED14.B, LED15.B, LED16.B
- net R3GREEN: now also LED13.G, LED14.G, LED15.G, LED16.G
- net R3RED: now also LED13.R, LED14.R, LED15.R, LED16.R
- net UNDGLOW: now also R12.2; no longer U$20.DIN
- net VCC: now also C18.2, C19.2, C20.2, C21.2, U$17.VDD, U$18.VDD, U$19.VDD, U$20.VDD
Other:
- note added: "RBG MATRIX"
- moved on the sheet: C1, C10, C11, C12, C13, C18, C19, C2, C20, C21, C6, C9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

Commit message: ESD protection, dxf board-switch matrix reference, started routing
Parts:
- removed LED1, LED10, LED11, LED12, LED13, LED14, LED15, LED16, LED2, LED3, LED4, LED5, LED6, LED7, LED8, LED9: 6028RGBLED_BOTTOM, 6028LED:6028RGBLED_BOTTOM
- removed U$17, U$18, U$19, U$20: SK6812MINI-E_BOTTOM, SK6812MINI-E:SK6812MINI-E_BOTTOM
- added F17: 1206L012, polyfuse-smd_10:1206L012
- added RGB1, RGB10, RGB11, RGB12, RGB13, RGB14, RGB15, RGB16, RGB2, RGB3, RGB4, RGB5, RGB6, RGB7, RGB8, RGB9: 6028RGBLED_BOTTOM, 6028LED:6028RGBLED_BOTTOM
- added U$1: PRTR5V0U2X, Controller:PRTR5V0U2X
- added UGLOW1, UGLOW2, UGLOW3, UGLOW4: SK6812MINI-E, SK6812MINI-E:SK6812MINI-E
Connections:
- new net VUSB: F17.2, J1.VBUS
- net 0: now also U$1.1, UGLOW1.GND, UGLOW2.GND, UGLOW3.GND, UGLOW4.GND; no longer U$17.GND, U$18.GND, U$19.GND, U$20.GND
- net C0RGB: now also RGB1.VIN, RGB13.VIN, RGB5.VIN, RGB9.VIN; no longer LED1.VIN, LED13.VIN, LED5.VIN, LED9.VIN
- net C1RGB: now also RGB10.VIN, RGB14.VIN, RGB2.VIN, RGB6.VIN; no longer LED10.VIN, LED14.VIN, LED2.VIN, LED6.VIN
- net C2RGB: now also RGB11.VIN, RGB15.VIN, RGB3.VIN, RGB7.VIN; no longer LED11.VIN, LED15.VIN, LED3.VIN, LED7.VIN
- net C3RGB: now also RGB12.VIN, RGB16.VIN, RGB4.VIN, RGB8.VIN; no longer LED12.VIN, LED16.VIN, LED4.VIN, LED8.VIN
- net D+: now also U$1.2
- net D-: now also U$1.3
- net N$25: now also UGLOW2.DOUT, UGLOW3.DIN; no longer U$18.DIN, U$19.DOUT
- net N$39: now also UGLOW1.DOUT, UGLOW2.DIN; no longer U$19.DIN, U$20.DOUT
- net N$6: now also UGLOW3.DOUT, UGLOW4.DIN; no longer U$17.DIN, U$18.DOUT
- net N$7: now also UGLOW1.DIN; no longer U$20.DIN
- net R0BLUE: now also RGB1.B, RGB2.B, RGB3.B, RGB4.B; no longer LED1.B, LED2.B, LED3.B, LED4.B
- net R0GREEN: now also RGB1.G, RGB2.G, RGB3.G, RGB4.G; no longer LED1.G, LED2.G, LED3.G, LED4.G
- net R0RED: now also RGB1.R, RGB2.R, RGB3.R, RGB4.R; no longer LED1.R, LED2.R, LED3.R, LED4.R
- net R1BLUE: now also RGB5.B, RGB6.B, RGB7.B, RGB8.B; no longer LED5.B, LED6.B, LED7.B, LED8.B
- net R1GREEN: now also RGB5.G, RGB6.G, RGB7.G, RGB8.G; no longer LED5.G, LED6.G, LED7.G, LED8.G
- net R1RED: now also RGB5.R, RGB6.R, RGB7.R, RGB8.R; no longer LED5.R, LED6.R, LED7.R, LED8.R
- net R2BLUE: now also RGB10.B, RGB11.B, RGB12.B, RGB9.B; no longer LED10.B, LED11.B, LED12.B, LED9.B
- net R2GREEN: now also RGB10.G, RGB11.G, RGB12.G, RGB9.G; no longer LED10.G, LED11.G, LED12.G, LED9.G
- net R2RED: now also RGB10.R, RGB11.R, RGB12.R, RGB9.R; no longer LED10.R, LED11.R, LED12.R, LED9.R
- net R3BLUE: now also RGB13.B, RGB14.B, RGB15.B, RGB16.B; no longer LED13.B, LED14.B, LED15.B, LED16.B
- net R3GREEN: now also RGB13.G, RGB14.G, RGB15.G, RGB16.G; no longer LED13.G, LED14.G, LED15.G, LED16.G
- net R3RED: now also RGB13.R, RGB14.R, RGB15.R, RGB16.R; no longer LED13.R, LED14.R, LED15.R, LED16.R
- net VCC: now also F17.1, U$1.4, UGLOW1.VDD, UGLOW2.VDD, UGLOW3.VDD, UGLOW4.VDD; no longer J1.VBUS, U$17.VDD, U$18.VDD, U$19.VDD, U$20.VDD
Other:
- note added: "ESD PROTECTION"
- moved on the sheet: C1, C10, C11, C12, C13, C15, C18, C19, C2, C20, C21, C3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
